File: 2026_bike_rear_light/rear_light/rear_light.kicad_sch (KiCad schematic)
At the start: 22 parts, among them J1 Conn_01x04, J2 Conn_01x05, Q1 2N5551, Q2 FQP27P06, Q3 IRL540N, Q4 FQP27P06, Q5 2N5551, Q6 2N5551, U1 LM2596HV

Commit message: Bike Rear Light - pcb layout
Parts:
- ATtiny85: footprint (none) -> Connector_PinHeader_1.00mm:PinHeader_1x06_P1.00mm_Vertical
- ATtiny85_pwr1: footprint (none) -> Connector_PinHeader_1.00mm:PinHeader_1x03_P1.00mm_Vertical
- D1, D2: footprint (none) -> LED_THT:LED_D3.0mm
- J1: footprint (none) -> Connector_PinHeader_1.00mm:PinHeader_1x04_P1.00mm_Vertical
- J2: footprint (none) -> Connector_PinHeader_1.00mm:PinHeader_1x05_P1.00mm_Vertical_SMD_Pin1Left
- R1, R2, R3, R4, R5, R6, R7, R8, R9: footprint (none) -> Resistor_THT:R_Axial_DIN0204_L3.6mm_D1.6mm_P1.90mm_Vertical
Connections:
- net +48V: now also J1.1 (Pin_1); no longer J1.3 (Pin_3)
- net +5V: now also J1.3 (Pin_3); no longer J1.1 (Pin_1)
- no-connect marks 2 -> 4
Changed lines of the file:
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@@
 	)
 	(no_connect
+		(at 63.5 52.07)
+	)
+	(no_connect
 		(at 99.06 133.35)
 	)
+	(no_connect
+		(at 63.5 41.91)
+	)
 	(wire
 		(pts
@@
 	(wire
 		(pts
-			(xy 156.21 44.45) (xy 156.21 49.53)
+			(xy 151.13 44.45) (xy 151.13 49.53)
 		)
 		(stroke
@@
 	(wire
 		(pts
-			(xy 151.13 44.45) (xy 151.13 49.53)
+			(xy 156.21 44.45) (xy 156.21 49.53)
 		)
 		(stroke
@@
 	)
 	(label "BATT"
-		(at 151.13 46.99 0)
+		(at 156.21 46.99 0)
 		(effects
 			(font
@@
 	)
 	(label "SYS"
-		(at 156.21 48.26 0)
+		(at 151.13 45.72 0)
 		(effects
 			(font
@@
 			)
 		)
-		(property "Footprint" ""
+		(property "Footprint" "Resistor_THT:R_Axial_DIN0204_L3.6mm_D1.6mm_P1.90mm_Vertical"
 			(at 69.85 117.348 90)
 			(effects
@@
 			)
 		)
-		(property "Footprint" ""
+		(property "Footprint" "Connector_PinHeader_1.00mm:PinHeader_1x06_P1.00mm_Vertical"
 			(at 58.42 46.99 0)
 			(effects
@@
 	(symbol
 		(lib_id "power:+5V")
-		(at 156.21 44.45 0)
+		(at 151.13 44.45 0)
 		(unit 1)
 		(exclude_from_sim no)
@@
 		(dnp no)
 		(property "Reference" "#PWR014"
-			(at 156.21 48.26 0)
+			(at 151.13 48.26 0)
 			(effects
 				(font
@@
 		)
 		(property "Value" "+5V"
-			(at 156.21 40.386 0)
+			(at 151.13 40.386 0)
 			(effects
 				(font
@@
 		)
 		(property "Footprint" ""
-			(at 156.21 44.45 0)
+			(at 151.13 44.45 0)
 			(effects
 				(font
@@
 		)
 		(property "Datasheet" ""
-			(at 156.21 44.45 0)
+			(at 151.13 44.45 0)
 			(effects
 				(font
@@
 		)
 		(property "Description" "Power symbol creates a global label with name \"+5V\""
-			(at 156.21 44.45 0)
+			(at 151.13 44.45 0)
 			(effects
 				(font
@@
 	(symbol
 		(lib_id "power:+48V")
-		(at 151.13 44.45 0)
+		(at 156.21 44.45 0)
 		(unit 1)
 		(exclude_from_sim no)
@@
 		(dnp no)
 		(property "Reference" "#PWR012"
-			(at 151.13 48.26 0)
+			(at 156.21 48.26 0)
 			(effects
 				(font
@@
 		)
 		(property "Value" "+48V"
-			(at 151.13 40.894 0)
+			(at 156.21 40.894 0)
 			(effects
 				(font
@@
 		)
 		(property "Footprint" ""
-			(at 151.13 44.45 0)
+			(at 156.21 44.45 0)
 			(effects
 				(font
@@
 		)
 		(property "Datasheet" ""
-			(at 151.13 44.45 0)
+			(at 156.21 44.45 0)
 			(effects
 				(font
@@
 		)
 		(property "Description" "Power symbol creates a global label with name \"+48V\""
-			(at 151.13 44.45 0)
+			(at 156.21 44.45 0)
 			(effects
 				(font
@@
 			)
 		)
-		(property "Footprint" ""
+		(property "Footprint" "Resistor_THT:R_Axial_DIN0204_L3.6mm_D1.6mm_P1.90mm_Vertical"
 			(at 62.23 123.698 90)
 			(effects
@@
 			)
 		)
-		(property "Footprint" ""
+		(property "Footprint" "Resistor_THT:R_Axial_DIN0204_L3.6mm_D1.6mm_P1.90mm_Vertical"
 			(at 36.83 136.398 90)
 			(effects
@@
 			)
 		)
-		(property "Footprint" ""
+		(property "Footprint" "Resistor_THT:R_Axial_DIN0204_L3.6mm_D1.6mm_P1.90mm_Vertical"
 			(at 152.4 123.698 90)
 			(effects
@@
 			)
 		)
-		(property "Footprint" ""
+		(property "Footprint" "Resistor_THT:R_Axial_DIN0204_L3.6mm_D1.6mm_P1.90mm_Vertical"
 			(at 159.258 118.11 90)
 			(effects
@@
 			)
 		)
-		(property "Footprint" ""
+		(property "Footprint" "Resistor_THT:R_Axial_DIN0204_L3.6mm_D1.6mm_P1.90mm_Vertical"
 			(at 137.922 119.38 90)
 			(effects
@@
 			)
 		)
-		(property "Footprint" ""
+		(property "Footprint" "Connector_PinHeader_1.00mm:PinHeader_1x04_P1.00mm_Vertical"
 			(at 153.67 54.61 0)
 			(effects
@@
 			)
 		)
-		(property "Footprint" ""
+		(property "Footprint" "LED_THT:LED_D3.0mm"
 			(at 238.76 118.11 0)
 			(effects
@@
 			)
 		)
-		(property "Footprint" ""
+		(property "Footprint" "Resistor_THT:R_Axial_DIN0204_L3.6mm_D1.6mm_P1.90mm_Vertical"
 			(at 36.83 116.078 90)
 			(effects
@@
 			)
 		)
-		(property "Footprint" ""
+		(property "Footprint" "Resistor_THT:R_Axial_DIN0204_L3.6mm_D1.6mm_P1.90mm_Vertical"
 			(at 224.282 134.62 90)
 			(effects
@@
 			)
 		)
-		(property "Footprint" ""
+		(property "Footprint" "LED_THT:LED_D3.0mm"
 			(at 170.18 133.35 0)
 			(effects
@@
 			)
 		)
-		(property "Footprint" ""
+		(property "Footprint" "Connector_PinHeader_1.00mm:PinHeader_1x03_P1.00mm_Vertical"
 			(at 45.72 50.8 0)
 			(effects
@@
 			)
 		)
-		(property "Footprint" ""
+		(property "Footprint" "Connector_PinHeader_1.00mm:PinHeader_1x05_P1.00mm_Vertical_SMD_Pin1Left"
 			(at 224.79 53.34 0)
 			(effects
@@
 			)
 		)
-		(property "Footprint" ""
+		(property "Footprint" "Resistor_THT:R_Axial_DIN0204_L3.6mm_D1.6mm_P1.90mm_Vertical"
 			(at 217.17 131.318 90)
 			(effects

Commit message: Rear Bike Light - Update schematic and PBC layout  - Remove the older brake light circuit  - Layout the PCB components (roughly)
Parts:
- removed Q3: IRL540N, Package_TO_SOT_THT:TO-220-3_Vertical, symbol Transistor_FET:IRF540N
- added Q3: 2N5551, Package_TO_SOT_THT:TO-92_Inline, symbol Transistor_BJT:PN2222A
- added Q7: FQP27P06, Package_TO_SOT_THT:TO-220-3_Vertical, symbol Transistor_FET:FQP27P06
- added R10, R11: 10k, Resistor_THT:R_Axial_DIN0204_L3.6mm_D1.6mm_P1.90mm_Vertical, symbol Device:R
- R4: value 300 -> 33k
- R5: value 100k -> 33k
Connections:
- net +48V: now also Q7.3 (S), R10.2; no longer D2.1 (K)
- net +5V: now also R11.2; no longer ATtiny85.4 (Pin_4)
- net BRAKE: now also Q7.2 (D)
- net GND: now also D2.1 (K), Q3.1 (E); no longer R5.2
- net at R4.2: now also Q3.2 (B); no longer R5.1
- new net: Q7.1 (G), R10.1, R5.2
- new net: Q3.3 (C), R5.1
- new net PB3: ATtiny85.4 (Pin_4), R11.1
Other:
- note removed: "DO NOT USE - Is a low side circuit"
